File: pcb/kaasch-keys-pbc-left.kicad_pcb (KiCad board)
At the start: 2 copper layers, 154.8 x 128.9 mm, 73 parts, among them J1 Conn_01x12_Pin, J2 Conn_01x12_Pin, SW1 SW_Push, SW10 SW_Push, SW11 SW_Push, SW12 SW_Push, SW13 SW_Push, SW14 SW_Push, SW15 SW_Push, SW16 SW_Push, SW17 SW_Push, SW18 SW_Push, SW19 SW_Push, SW2 SW_Push, SW20 SW_Push, SW21 SW_Push, SW22 SW_Push, SW23 SW_Push, SW24 SW_Push, SW25 SW_Push, SW26 SW_Push, SW27 SW_Push, SW28 SW_Push, SW29 SW_Push, SW3 SW_Push, SW30 SW_Push, SW31 SW_Push, SW32 SW_Push, SW33 SW_Push, SW34 SW_Push, SW35 SW_Push, SW36 SW_Push_Reset, SW4 SW_Push, SW5 SW_Push, SW6 SW_Push, SW7 SW_Push, SW8 SW_Push, SW9 SW_Push

Commit message: swaggers
Parts:
- moved J1 15.2 mm to (227.4, 38.1)
- moved J2 15.2 mm to (212.2, 38.1)
- moved D1 1.07 mm to (85.2, 47.5)
- moved D2 1.07 mm to (85.2, 66.5)
- moved D7 1.07 mm to (104.1, 66.5)
- moved D8 1.07 mm to (104.2, 85.5)
- moved D35 1.04 mm to (216.5, 152.4)
- moved D6 1.03 mm to (104.3, 47.5)
- moved D3 1.01 mm to (85.2, 85.6)
- moved D11 1.00 mm to (123.3, 47.5)
- moved D4 0.98 mm to (85.2, 104.7)
- moved D16 0.96 mm to (142.4, 47.5)
- moved D12 0.96 mm to (123.3, 66.6)
- moved D5 0.95 mm to (85.2, 123.7)
- moved D9 0.94 mm to (104.3, 104.7)
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Routing:
- net col.5.L: track 162.3 -> 114.4 mm, vias 0 -> 2
- net col.4.L: track 169.0 -> 122.5 mm, vias 2 -> 4
- net col.3.L: track 187.4 -> 147.4 mm, vias 2 -> 6
- net col.1.L: track 221.6 -> 182.4 mm, vias 2 -> 10
- net col.2.L: track 204.0 -> 164.9 mm, vias 2 -> 8
- net col.0.L: track 238.5 -> 200.9 mm, vias 2 -> 12
- net col.6.L: track 172.4 -> 135.3 mm
- net row.0.L: track 146.6 -> 178.6 mm, vias 0 -> 2
- net row.1.L: track 134.3 -> 165.8 mm, vias 0 -> 2
- net row.4.L: track 253.7 -> 264.7 mm, vias 2 -> 0
- net Net-(J2-Pin_3): track 77.8 -> 66.9 mm, vias 1 -> 0
- net row.2.L: track 185.7 -> 180.3 mm
- net row.3.L: track 232.1 -> 235.9 mm
- net Net-(D35-A): track 7.44 -> 6.65 mm, vias 1 -> 0
- net Net-(D30-A): track 7.48 -> 6.75 mm, vias 1 -> 0
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
Commit message: continue on design
Parts:
- added J3: Conn_JST, Connector_JST:JST_EH_B2B-EH-A_1x02_P2.50mm_Vertical, F.Cu at (227.4, 76.2)
- added SW37: SW_Slide_Bat, Button_Switch_SMD:SW_SPDT_PCM12, F.Cu at (219.8, 41.2)
Connections:
- J2 pad 1: unconnected-(J2-Pin_1-Pad1) -> RAW
Routing:
- net BAT+: track 0.00 -> 36.0 mm
- net RAW: track 0.00 -> 11.0 mm
