File: pcb/kaasch-keys-pcb-right.kicad_pcb (KiCad board)
At the start: 2 copper layers, 154.8 x 128.9 mm, 73 parts, among them J1 Conn_01x12_Pin, J2 Conn_01x12_Pin, SW1 SW_Push, SW10 SW_Push, SW11 SW_Push, SW12 SW_Push, SW13 SW_Push, SW14 SW_Push, SW15 SW_Push, SW16 SW_Push, SW17 SW_Push, SW18 SW_Push, SW19 SW_Push, SW2 SW_Push, SW20 SW_Push, SW21 SW_Push, SW22 SW_Push, SW23 SW_Push, SW24 SW_Push, SW25 SW_Push, SW26 SW_Push, SW27 SW_Push, SW28 SW_Push, SW29 SW_Push, SW3 SW_Push, SW30 SW_Push, SW31 SW_Push, SW32 SW_Push, SW33 SW_Push, SW34 SW_Push, SW35 SW_Push, SW36 SW_Push_Reset, SW4 SW_Push, SW5 SW_Push, SW6 SW_Push, SW7 SW_Push, SW8 SW_Push, SW9 SW_Push

Commit message: swaggers
Parts:
- SW10, SW4: footprint Button_Switch_Keyboard:SW_Cherry_MX_1.00u_PCB -> Button_Switch_Keyboard:SW_Cherry_MX_1.50u_PCB
- moved SW4 223.0 mm to (106.2, 143.9), turned to -65 degrees
- moved SW1 180.6 mm to (106.2, 44.3)
- moved SW11 180.6 mm to (144.3, 44.3)
- moved SW12 180.6 mm to (144.3, 63.4)
- moved SW13 180.6 mm to (144.3, 82.4)
- moved SW14 180.6 mm to (144.3, 101.5)
- moved SW16 180.6 mm to (163.3, 44.3)
- moved SW17 180.6 mm to (163.3, 63.4)
- moved SW18 180.6 mm to (163.3, 82.4)
- moved SW19 180.6 mm to (163.3, 101.5)
- moved SW2 180.6 mm to (106.2, 63.4)
- moved SW20 180.6 mm to (163.3, 120.5)
- moved SW21 180.6 mm to (182.4, 44.3)
- moved SW22 180.6 mm to (182.4, 63.4)
- moved SW23 180.6 mm to (182.4, 82.4)
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Routing:
- net row.4.R: track 0.00 -> 150.6 mm
- net row.3.R: track 0.00 -> 144.4 mm
- net col.0.R: track 0.00 -> 124.6 mm
- net row.1.R: track 0.00 -> 120.8 mm
- net row.0.R: track 0.00 -> 120.1 mm
- net row.2.R: track 0.00 -> 120.1 mm
- net col.1.R: track 0.00 -> 92.2 mm
- net col.6.R: track 0.00 -> 76.2 mm
- net col.5.R: track 0.00 -> 76.2 mm
- net col.4.R: track 0.00 -> 76.2 mm
- net col.3.R: track 0.00 -> 76.2 mm
- net col.2.R: track 0.00 -> 76.2 mm
- net Net-(D5-A): track 0.00 -> 6.79 mm
- net Net-(D4-A): track 0.00 -> 6.78 mm
- net Net-(D10-A): track 0.00 -> 6.74 mm
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
Commit message: continue on design
Parts:
- added J3: Conn_JST, Connector_JST:JST_EH_B2B-EH-A_1x02_P2.50mm_Vertical, F.Cu at (78.9, 84.3)
- added SW37: SW_Slide_Bat, Button_Switch_SMD:SW_SPDT_PCM12, F.Cu at (86.5, 46.7)
Connections:
- J2 pad 1: unconnected-(J2-Pin_1-Pad1) -> RAW
Routing:
- net col.6.R: track 76.2 -> 234.9 mm
- net col.5.R: track 76.2 -> 210.3 mm, vias 0 -> 2
- net col.4.R: track 76.2 -> 190.9 mm, vias 0 -> 2
- net col.3.R: track 76.2 -> 181.1 mm, vias 0 -> 1
- net row.4.R: track 150.6 -> 245.6 mm, vias 0 -> 2
- net Net-(J2-Pin_3): track 0.00 -> 70.9 mm, vias 0 -> 4
- net row.3.R: track 144.4 -> 213.6 mm
- net col.2.R: track 76.2 -> 142.7 mm, vias 0 -> 3
- net col.1.R: track 92.2 -> 154.4 mm, vias 0 -> 3
- net col.0.R: track 124.6 -> 176.9 mm, vias 0 -> 3
- net BAT+: track 0.00 -> 40.7 mm, vias 0 -> 1
- net row.2.R: track 120.1 -> 153.1 mm
- net row.0.R: track 120.1 -> 137.6 mm, vias 0 -> 1
- net row.1.R: track 120.8 -> 135.2 mm, vias 0 -> 1
- net RAW: track 0.00 -> 11.7 mm

Commit message: gerberz for testing export config, ready for 3d print testing
Routing:
- net Net-(D20-A): track 0.00 -> 6.54 mm
- net Net-(D15-A): track 0.00 -> 6.54 mm
- net col.1.R: track 154.4 -> 158.2 mm
- net Net-(D4-A): track 6.78 -> 7.32 mm

Commit message: moore
Connections:
- SW37 pad 1: BAT+ -> unconnected-(SW37-A-Pad1)
- SW37 pad 3: unconnected-(SW37-C-Pad3) -> BAT+
Routing:
- net BAT+: track 40.7 -> 38.9 mm
