File: pcb/left/pcb-left.kicad_pcb (KiCad board)
At the start: 2 copper layers, 154.8 x 128.9 mm, 75 parts, among them J1 Conn_01x12_Pin, J2 Conn_01x12_Pin, J3 Conn_JST, SW1 SW_Push, SW10 SW_Push, SW11 SW_Push, SW12 SW_Push, SW13 SW_Push, SW14 SW_Push, SW15 SW_Push, SW16 SW_Push, SW17 SW_Push, SW18 SW_Push, SW19 SW_Push, SW2 SW_Push, SW20 SW_Push, SW21 SW_Push, SW22 SW_Push, SW23 SW_Push, SW24 SW_Push, SW25 SW_Push, SW26 SW_Push, SW27 SW_Push, SW28 SW_Push, SW29 SW_Push, SW3 SW_Push, SW30 SW_Push, SW31 SW_Push, SW32 SW_Push, SW33 SW_Push, SW34 SW_Push, SW35 SW_Push, SW36 SW_Push_Reset, SW37 SW_Slide_Bat, SW4 SW_Push, SW5 SW_Push, SW6 SW_Push, SW7 SW_Push, SW8 SW_Push, SW9 SW_Push

Commit message: changes 2
Parts:
- J3: footprint Connector_JST:JST_EH_B2B-EH-A_1x02_P2.50mm_Vertical -> Connector_JST:JST_PH_S2B-PH-K_1x02_P2.00mm_Horizontal
- moved J3 5.99 mm to (230.6, 81.3)
- moved SW37 3.99 mm to (223.0, 38.8)
- moved J1 3.17 mm to (230.6, 38.1)
- moved J2 3.17 mm to (215.4, 38.1)
Routing:
- net BAT+: track 36.0 -> 47.6 mm
- net row.0.L: track 178.6 -> 183.4 mm
- net row.1.L: track 165.8 -> 169.9 mm
- net row.2.L: track 180.3 -> 183.9 mm
- net col.4.L: track 122.5 -> 125.6 mm
- net row.3.L: track 235.9 -> 239.0 mm
- net col.5.L: track 114.4 -> 117.3 mm
- net row.4.L: track 264.7 -> 267.2 mm
- net col.1.L: track 182.4 -> 184.3 mm
- net col.0.L: track 200.9 -> 202.7 mm
- net RAW: track 11.0 -> 12.4 mm
- net Net-(J2-Pin_3): track 66.9 -> 65.6 mm
- net col.2.L: track 164.9 -> 166.0 mm
- net col.6.L: track 135.3 -> 135.8 mm
Other:
- outline, holes or cut-outs redrawn

Commit message: added stls
Parts:
- J1, J2: moved to F.Cu
- turned J1 to 0 degrees
- turned J2 to 0 degrees
