File: pcb/right/pcb-right.kicad_pcb (KiCad board)
At the start: 2 copper layers, 154.8 x 128.9 mm, 75 parts, among them J1 Conn_01x12_Pin, J2 Conn_01x12_Pin, J3 Conn_JST, SW1 SW_Push, SW10 SW_Push, SW11 SW_Push, SW12 SW_Push, SW13 SW_Push, SW14 SW_Push, SW15 SW_Push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

Commit message: pcb corrections
Parts:
- J3: footprint Connector_JST:JST_EH_B2B-EH-A_1x02_P2.50mm_Vertical -> Connector_JST:JST_PH_B2B-PH-K_1x02_P2.00mm_Vertical
- moved J3 0.50 mm to (78.9, 83.8)
