File: pcb/right/pcb-right.kicad_pcb (KiCad board)
At the start: 2 copper layers, 154.8 x 128.9 mm, 75 parts, among them J1 Conn_01x12_Pin, J2 Conn_01x12_Pin, J3 Conn_JST, SW1 SW_Push, SW10 SW_Push, SW11 SW_Push, SW12 SW_Push, SW13 SW_Push, SW14 SW_Push, SW15 SW_Push, SW16 SW_Push, SW17 SW_Push, SW18 SW_Push, SW19 SW_Push, SW2 SW_Push, SW20 SW_Push, SW21 SW_Push, SW22 SW_Push, SW23 SW_Push, SW24 SW_Push, SW25 SW_Push, SW26 SW_Push, SW27 SW_Push, SW28 SW_Push, SW29 SW_Push, SW3 SW_Push, SW30 SW_Push, SW31 SW_Push, SW32 SW_Push, SW33 SW_Push, SW34 SW_Push, SW35 SW_Push, SW36 SW_Push_Reset, SW37 SW_Slide_Bat, SW4 SW_Push, SW5 SW_Push, SW6 SW_Push, SW7 SW_Push, SW8 SW_Push, SW9 SW_Push

Commit message: changes 2
Parts:
- J3: footprint Connector_JST:JST_EH_B2B-EH-A_1x02_P2.50mm_Vertical -> Connector_JST:JST_PH_S2B-PH-K_1x02_P2.00mm_Horizontal
- moved J3 5.57 mm to (75.7, 88.9)
- moved SW37 3.99 mm to (83.3, 44.3)
- moved J2 3.18 mm to (75.7, 43.7)
- moved J1 3.17 mm to (90.9, 43.7)
Routing:
- net col.2.R: track 142.7 -> 163.2 mm
- net BAT+: track 38.9 -> 45.3 mm
- net Net-(J2-Pin_3): track 70.9 -> 77.4 mm, vias 4 -> 1
- net row.1.R: track 135.2 -> 138.4 mm
- net row.2.R: track 153.1 -> 156.2 mm
- net row.0.R: track 137.6 -> 140.8 mm
- net col.5.R: track 210.3 -> 213.1 mm
- net col.4.R: track 190.9 -> 193.0 mm
- net col.1.R: track 158.2 -> 159.9 mm
- net row.4.R: track 245.6 -> 244.0 mm
- net col.6.R: track 234.9 -> 233.5 mm
- net RAW: track 11.7 -> 12.7 mm
- net col.3.R: track 181.1 -> 182.0 mm
- net row.3.R: track 213.6 -> 214.4 mm
- net col.0.R: track 176.9 -> 177.2 mm, vias 3 -> 5
Other:
- outline, holes or cut-outs redrawn

Commit message: added stls
Parts:
- J1, J2: moved to F.Cu
- turned J1 to 0 degrees
- turned J2 to 0 degrees
Routing:
- net BAT+: track 45.3 -> 46.3 mm
